File: main/b1.kicad_sch (KiCad schematic)
At the start: 37 parts, among them J1 Micro_SD_Card_Det1, J10 STKHEADER_B1_R, J11 STKHEADER_B1_L, J2 HEADER_ST-Link IN, J4 7.4V_IN, J5 Voltmeter_OUT, J6 SCRTERM_Board3ConnPt, U2 LSM6DSL, U3 MMC5883MA, U4 AP63203WU, U5 THVD1420D

Commit message: work on dsn checklist
Parts:
- removed C22: 100n, Capacitor_SMD:C_0603_1608Metric, symbol Device:C
- removed U5: THVD1420D, Package_SO:SOIC-8_3.9x4.9mm_P1.27mm, symbol Interface_UART:THVD1420D
- added Q1: AO3401A, Package_TO_SOT_SMD:SOT-23, symbol Transistor_FET:AO3401A
- added R18: 10k, Resistor_SMD:R_0603_1608Metric, symbol Device:R
- added U5: SP3485EN, Package_SO:SOIC-8_3.9x4.9mm_P1.27mm, symbol Interface_UART:SP3485EN
- L1: footprint Inductor_SMD:L_0603_1608Metric -> Inductor_SMD:L_6.3x6.3_H3
- U6: footprint Oscillator:Oscillator_SMD_SCTF_SX3M8.000M20F30TNN -> Crystal:Crystal_SMD_3225-4Pin_3.2x2.5mm
Connections:
- net +3V3: now also U5.8 (VCC); no longer U6.4 (VDD)
- net B1_RS485_MODE_SW: now also U5.2 (~{RE}), U5.3 (DE)
- net B1_RS485_RX: now also U5.4 (DI)
- net B1_RS485_TX: now also U5.1 (RO)
- net BAT_+: now also Q1.3 (D); no longer C16.1, U4.2 (EN), U4.3 (IN)
- net GND: now also U6.4 (GND), R18.1, U5.5 (GND)
- net at R2.1: now also U5.6 (A)
- net at R3.1: now also U5.7 (B)
- net MCU_OSC_OUT: now reaches U6.1 (OSCIN)
- new net: C16.1, Q1.2 (S), U4.2 (EN), U4.3 (IN)
- new net: Q1.1 (G), R18.2
- no-connect marks 3 -> 2
Other:
- moved on the sheet: C16, C17, C18, C21, L1, U4

Commit message: continue fixing chklst
Parts:
- added R20: 10k, Resistor_SMD:R_0603_1608Metric, symbol Device:R_Small
Connections:
- net +3V3: now also R20.1
- net GND: now also J1.SH (SHIELD)
- net SDIO_CMD: now also R20.2
- no-connect marks 2 -> 1
Other:
- moved on the sheet: C28

Commit message: prep gerber and cpl/bom
Parts:
- added C47, C48: 10p, Capacitor_SMD:C_0603_1608Metric, symbol Device:C
- C16: value 10u -> 10u 25V; footprint Capacitor_SMD:C_0603_1608Metric -> Capacitor_SMD:C_0805_2012Metric; LCSC (none) -> C15850
- C18, C21: LCSC (none) -> C59461
- D1: value LED -> LED red; LCSC (none) -> C84256
- J10, J11, J2, J4, J5, J6: now not fitted; now left out of the parts list
- Q1: LCSC (none) -> C15127
- R6, R7: value 4.7k -> 2.7k
- R8: value 10k -> 1k
- U3: value MMC5883MA -> MMC5983MA
- U5: LCSC (none) -> C8963
- U6: value (none) -> 16MHz; LCSC (none) -> C13738; MPN (none) -> YXC X322516MLB4SI
Connections:
- net +3V3: now also U3.4 (I2C_SEL)
- net GND: now also C47.2, C48.2
- net MCU_OSC_IN: now also C47.1
- net MCU_OSC_OUT: now also C48.1
Other:
- note added: "Crystal load caps for U6: 10 pF C0G, place within 2 mm of the crystal"
- moved on the sheet: U6
