File: main/b2.kicad_sch (KiCad schematic)
At the start: 15 parts, among them J12 STKHEADER_B2_R, J7 HEADER_ST-Link IN, J9 STKHEADER_B2_L, U12 BMI323

Commit message: work on dsn checklist
Parts:
- removed C33: 100n, Capacitor_SMD:C_0603_1608Metric, symbol Device:C
- U11: footprint Oscillator:Oscillator_SMD_SCTF_SX3M8.000M20F30TNN -> Crystal:Crystal_SMD_3225-4Pin_3.2x2.5mm
Connections:
- net B_VDDIO is gone; now on net +3V3: C35.1, U12.5 (VDDIO)
- net +3V3: no longer U11.4 (VDD)
- net GND: now also U11.4 (GND)
- net MCU_OSC_OUT: now reaches U11.1 (OSCIN)
- no-connect marks 2 -> 1
Changed lines of the file:
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@@
+	)
+	(junction
+		(at 29.21 93.98)
+		(diameter 0)
+		(color 0 0 0 0)
 	)
 	(junction
@@
 	)
 	(junction
-		(at 67.31 39.37)
-		(diameter 0)
-		(color 0 0 0 0)
-	)
-	(junction
 		(at 134.62 60.96)
 		(diameter 0)
@@
 		(at 124.46 33.02)
 	)
-	(no_connect
-		(at 48.26 39.37)
-	)
 	(wire
 		(pts
-			(xy 24.13 93.98) (xy 43.18 93.98)
+			(xy 24.13 93.98) (xy 29.21 93.98)
 		)
 		(stroke
@@
 	(wire
 		(pts
-			(xy 66.04 41.91) (xy 78.74 41.91)
+			(xy 134.62 68.58) (xy 139.7 68.58)
 		)
 		(stroke
@@
 	(wire
 		(pts
-			(xy 134.62 68.58) (xy 139.7 68.58)
+			(xy 85.09 99.06) (xy 83.82 99.06)
 		)
 		(stroke
@@
 	(wire
 		(pts
-			(xy 85.09 99.06) (xy 83.82 99.06)
+			(xy 41.91 99.06) (xy 41.91 96.52)
 		)
 		(stroke
@@
 	(wire
 		(pts
-			(xy 41.91 99.06) (xy 41.91 96.52)
+			(xy 146.05 63.5) (xy 146.05 68.58)
 		)
 		(stroke
@@
 	(wire
 		(pts
-			(xy 146.05 63.5) (xy 146.05 68.58)
+			(xy 40.64 99.06) (xy 41.91 99.06)
 		)
 		(stroke
@@
 	(wire
 		(pts
-			(xy 40.64 99.06) (xy 41.91 99.06)
+			(xy 129.54 60.96) (xy 134.62 60.96)
 		)
 		(stroke
@@
 	(wire
 		(pts
-			(xy 129.54 60.96) (xy 134.62 60.96)
+			(xy 52.07 110.49) (xy 60.96 110.49)
 		)
 		(stroke
@@
 	(wire
 		(pts
-			(xy 52.07 110.49) (xy 60.96 110.49)
+			(xy 41.91 96.52) (xy 43.18 96.52)
 		)
 		(stroke
@@
 	(wire
 		(pts
-			(xy 41.91 96.52) (xy 43.18 96.52)
+			(xy 139.7 68.58) (xy 146.05 68.58)
 		)
 		(stroke
@@
 	(wire
 		(pts
-			(xy 139.7 68.58) (xy 146.05 68.58)
+			(xy 29.21 93.98) (xy 43.18 93.98)
 		)
 		(stroke
@@
 	(wire
 		(pts
-			(xy 146.05 68.58) (xy 160.02 68.58)
+			(xy 29.21 93.98) (xy 29.21 99.06)
 		)
 		(stroke
@@
 	(wire
 		(pts
-			(xy 34.29 110.49) (xy 44.45 110.49)
+			(xy 146.05 68.58) (xy 160.02 68.58)
 		)
 		(stroke
@@
 	(wire
 		(pts
-			(xy 160.02 68.58) (xy 160.02 63.5)
+			(xy 34.29 110.49) (xy 44.45 110.49)
 		)
 		(stroke
@@
 	(wire
 		(pts
-			(xy 138.43 92.71) (xy 144.78 92.71)
+			(xy 160.02 68.58) (xy 160.02 63.5)
 		)
 		(stroke
@@
 	(wire
 		(pts
-			(xy 67.31 39.37) (xy 74.93 39.37)
+			(xy 138.43 92.71) (xy 144.78 92.71)
 		)
 		(stroke
@@
 	(wire
 		(pts
-			(xy 29.21 99.06) (xy 29.21 93.98)
+			(xy 67.31 39.37) (xy 66.04 39.37)
 		)
 		(stroke
@@
 		)
 	)
-	(wire
-		(pts
-			(xy 67.31 39.37) (xy 66.04 39.37)
-		)
-		(stroke
-			(width 0)
-			(type default)
-		)
-	)
 	(label "B_GNDIO"
 		(at 60.96 110.49 180)
@@
 		)
 	)
-	(hierarchical_label "MCU_OSC_IN"
-		(shape output)
-		(at 78.74 41.91 0)
-		(effects
-			(font
-				(size 1.27 1.27)
-			)
-			(justify left)
-		)
-	)
 	(hierarchical_label "B2_MISO"
 		(shape output)
@@
 		)
 	)
+	(hierarchical_label "MCU_OSC_IN"
+		(shape output)
+		(at 66.04 41.91 0)
+		(effects
+			(font
+				(size 1.27 1.27)
+			)
+			(justify left)
+		)
+	)
 	(hierarchical_label "BMI_MOSI"
 		(shape input)
@@
 			)
 			(justify left)
+		)
+	)
+	(hierarchical_label "MCU_OSC_OUT"
+		(shape input)
+		(at 48.26 39.37 180)
+		(effects
+			(font
+				(size 1.27 1.27)
+			)
+			(justify right)
 		)
 	)
@@
 		(in_pos_files yes)
 		(dnp no)
-		(fields_autoplaced yes)
 		(property "Reference" "#PWR065"
 			(at 29.21 95.25 0)
@@
 	)
 	(symbol
-		(lib_id "Device:C")
-		(at 67.31 35.56 0)
-		(unit 1)
-		(body_style 1)
-		(exclude_from_sim no)
-		(in_bom yes)
-		(on_board yes)
-		(in_pos_files yes)
-		(dnp no)
-		(property "Reference" "C33"
-			(at 70.104 34.29 0)
-			(show_name no)
-			(do_not_autoplace no)
-			(effects
-				(font
-					(size 1.27 1.27)
-				)
-				(justify left)
-			)
-		)
-		(property "Value" "100n"
-			(at 70.104 36.83 0)
-			(show_name no)
-			(do_not_autoplace no)
-			(effects
-				(font
-					(size 1.27 1.27)
-				)
-				(justify left)
-			)
-		)
-		(property "Footprint" "Capacitor_SMD:C_0603_1608Metric"
-			(at 68.2752 39.37 0)
-			(hide yes)
-			(show_name no)
-			(do_not_autoplace no)
-			(effects
-				(font
-					(size 1.27 1.27)
-				)
-			)
-		)
-		(property "Datasheet" ""
-			(at 67.31 35.56 0)
-			(hide yes)
-			(show_name no)
-			(do_not_autoplace no)
-			(effects
-				(font
-					(size 1.27 1.27)
-				)
-			)
-		)
-		(property "Description" "Unpolarized capacitor"
-			(at 67.31 35.56 0)
-			(hide yes)
-			(show_name no)
-			(do_not_autoplace no)
-			(effects
-				(font
-					(size 1.27 1.27)
-				)
-			)
-		)
-		(pin "1"
-		)
-		(pin "2"
-		)
-		(instances
-			(project "main"
-				(path "/6aa21aac-e8da-46e9-ae7a-f048cdfa6a26/59d03ad0-5707-4a1e-8261-79210a859241"
-					(reference "C33")
-					(unit 1)
-				)
-			)
-		)
-	)
-	(symbol
 		(lib_id "Connector_Generic:Conn_01x08")
 		(at 154.94 53.34 0)
@@
 			)
 		)
-		(property "Footprint" "Oscillator:Oscillator_SMD_SCTF_SX3M8.000M20F30TNN"
+		(property "Footprint" "Crystal:Crystal_SMD_3225-4Pin_3.2x2.5mm"
 			(at 57.15 40.64 0)
 			(hide yes)
@@
 	(symbol
 		(lib_id "power:GND")
-		(at 67.31 31.75 0)
+		(at 67.31 39.37 0)
 		(mirror x)
 		(unit 1)
@@
 		(dnp no)
 		(property "Reference" "#PWR061"
-			(at 67.31 25.4 0)
+			(at 67.31 33.02 0)
 			(hide yes)
 			(show_name no)
@@
 		)
 		(property "Value" "GND"
-			(at 67.31 26.67 0)
+			(at 67.31 34.29 0)
 			(show_name no)
 			(do_not_autoplace no)
@@
 		)
 		(property "Footprint" ""
-			(at 67.31 31.75 0)
+			(at 67.31 39.37 0)
 			(hide yes)
 			(show_name no)
@@
 		)
 		(property "Datasheet" ""
-			(at 67.31 31.75 0)
+			(at 67.31 39.37 0)
 			(hide yes)
 			(show_name no)
@@
 		)
 		(property "Description" "Power symbol creates a global label with name \"GND\" , ground"
-			(at 67.31 31.75 0)
+			(at 67.31 39.37 0)
 			(hide yes)
 			(show_name no)
@@
 					(unit 1)
 				)
-			)
-		)
-	)
-	(symbol
-		(lib_id "power:+3V3")
-		(at 74.93 39.37 270)
-		(unit 1)
-		(body_style 1)
-		(exclude_from_sim no)
-		(in_bom yes)
-		(on_board yes)
-		(in_pos_files yes)
-		(dnp no)
-		(property "Reference" "#PWR063"
-			(at 71.12 39.37 0)
-			(hide yes)
-			(show_name no)
-			(do_not_autoplace no)
-			(effects
-				(font
-					(size 1.27 1.27)
-				)
-			)
-		)
-		(property "Value" "+3V3"
-			(at 77.47 38.608 90)
-			(show_name no)
-			(do_not_autoplace no)
-			(effects
-				(font
-					(size 1.27 1.27)
-				)
-				(justify left)
-			)
-		)
-		(property "Footprint" ""
-			(at 74.93 39.37 0)
-			(hide yes)
-			(show_name no)
-			(do_not_autoplace no)
-			(effects
-				(font
-					(size 1.27 1.27)
-				)
-			)
-		)
-		(property "Datasheet" ""
-			(at 74.93 39.37 0)
-			(hide yes)
-			(show_name no)
-			(do_not_autoplace no)
-			(effects
-				(font
-					(size 1.27 1.27)
-				)
-			)
-		)
-		(property "Description" "Power symbol creates a global label with name \"+3V3\""
-			(at 74.93 39.37 0)
-			(hide yes)
-			(show_name no)
-			(do_not_autoplace no)
-			(effects
-				(font
-					(size 1.27 1.27)
-				)
-			)
-		)
-		(pin "1"
-		)
-		(instances
-			(project "main"
-				(path "/6aa21aac-e8da-46e9-ae7a-f048cdfa6a26/59d03ad0-5707-4a1e-8261-79210a859241"
-					(reference "#PWR063")
-					(unit 1)
-				)

Commit message: continue fixing chklst
Changed lines of the file:
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@@
 	)
 	(hierarchical_label "GPIO_D"
-		(shape bidirectional)
+		(shape output)
 		(at 160.02 55.88 0)
 		(effects
@@
 	)
 	(hierarchical_label "GPIO_B"
-		(shape bidirectional)
+		(shape output)
 		(at 160.02 50.8 0)
 		(effects
@@
 	)
 	(hierarchical_label "GPIO_E"
-		(shape bidirectional)
+		(shape output)
 		(at 160.02 58.42 0)
 		(effects
@@
 	)
 	(hierarchical_label "GPIO_A"
-		(shape bidirectional)
+		(shape output)
 		(at 160.02 48.26 0)
 		(effects
@@
 	)
 	(hierarchical_label "GPIO_C"
-		(shape bidirectional)
+		(shape output)
 		(at 160.02 53.34 0)
 		(effects

Commit message: prep gerber and cpl/bom
Parts:
- added C49, C50: 10p, Capacitor_SMD:C_0603_1608Metric, symbol Device:C
- D2: value LED -> LED red; LCSC (none) -> C84256
- J12, J9: footprint Connector_PinHeader_2.54mm:PinHeader_1x08_P2.54mm_Vertical -> Connector_PinSocket_2.54mm:PinSocket_1x08_P2.54mm_Vertical; now not fitted; now left out of the parts list
- J7: now not fitted; now left out of the parts list
- R14: value 10k -> 1k
- U11: value (none) -> 16MHz; LCSC (none) -> C13738; MPN (none) -> YXC X322516MLB4SI
Connections:
- net GND: now also C49.2, C50.2
- net MCU_OSC_IN: now also C49.1
- net MCU_OSC_OUT: now also C50.1
Other:
- note added: "Crystal load caps for U11: 10 pF C0G, place within 2 mm of the crystal"
