File: main/b3.kicad_sch (KiCad schematic)
At the start: 28 parts, among them J13 SCRTERM_Board3ConnPt, J8 HEADER_ST-Link IN, U13 MAX-M10S, U9 THVD1420D

Commit message: work on dsn checklist
Parts:
- removed C31: 100n, Capacitor_SMD:C_0603_1608Metric, symbol Device:C
- removed U9: THVD1420D, Package_SO:SOIC-8_3.9x4.9mm_P1.27mm, symbol Interface_UART:THVD1420D
- added U9: SP3485EN, Package_SO:SOIC-8_3.9x4.9mm_P1.27mm, symbol Interface_UART:SP3485EN
- U10: footprint Oscillator:Oscillator_SMD_SCTF_SX3M8.000M20F30TNN -> Crystal:Crystal_SMD_3225-4Pin_3.2x2.5mm
Connections:
- net +3V3: now also U9.8 (VCC); no longer U10.4 (VDD)
- net B3_RS485_MODE_SW: now also U9.2 (~{RE}), U9.3 (DE)
- net B3_RS485_RX: now also U9.4 (DI)
- net B3_RS485_TX: now also U9.1 (RO)
- net GND: now also U10.4 (GND), U9.5 (GND)
- net at R11.1: now also U9.6 (A)
- net at R12.1: now also U9.7 (B)
- net MCU_OSC_OUT: now reaches U10.1 (OSCIN)
- no-connect marks 6 -> 5

Commit message: continue fixing chklst
Parts:
- U13: now not fitted
Connections:
- net GPS_SAFEBOOT: no longer names the net of U13.18 (~{SAFEBOOT})
- no-connect marks 5 -> 6
Changed lines of the file:
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@@
+	)
+	(no_connect
+		(at 46.99 124.46)
 	)
 	(no_connect
@@
 			)
 			(justify left)
-		)
-	)
-	(hierarchical_label "GPS_SAFEBOOT"
-		(shape input)
-		(at 46.99 124.46 180)
-		(effects
-			(font
-				(size 1.27 1.27)
-			)
-			(justify right)
 		)
 	)
@@
 		(on_board yes)
 		(in_pos_files yes)
-		(dnp no)
+		(dnp yes)
 		(fields_autoplaced yes)
 		(property "Reference" "U13"

Commit message: prep gerber and cpl/bom
Parts:
- added C51, C52: 10p, Capacitor_SMD:C_0603_1608Metric, symbol Device:C
- added TP1: GPS_SAFEBOOT, TestPoint:TestPoint_Pad_D1.0mm, symbol Connector:TestPoint
- added TP4: GND, TestPoint:TestPoint_Pad_D1.0mm, symbol Connector:TestPoint
- AE1, J13, J8: now not fitted; now left out of the parts list
- D3: value LED -> LED red; LCSC (none) -> C84256
- L2: footprint Inductor_SMD:L_0402_1005Metric -> Inductor_SMD:L_0603_1608Metric
- R15: value 10k -> 1k
- U10: value (none) -> 16MHz; LCSC (none) -> C13738; MPN (none) -> YXC X322516MLB4SI
- U13: now left out of the parts list
- U9: LCSC (none) -> C8963
Connections:
- net GND: now also C51.2, C52.2, TP4.1
- net MCU_OSC_IN: now also C51.1
- net MCU_OSC_OUT: now also C52.1
- net GPS_SAFEBOOT: now reaches U13.18 (~{SAFEBOOT})
- net GPS_SAFEBOOT: now also TP1.1
- no-connect marks 6 -> 5
Other:
- note added: "Crystal load caps for U10: 10 pF C0G, place within 2 mm of the crystal"
- note added: "GPS recovery: short SAFEBOOT to GND at power-up, then use TXD/RXD at 9600 baud"
