File: main/main.kicad_sch (KiCad schematic)
At the start: 21 parts, among them U1 STM32F405RGTx, U7 STM32G071CBT6, U8 STM32G071CBT6

Commit message: work on dsn checklist
Connections:
- net B2_OSC_OUT: now reaches U7.9 (PF1-OSC_OUT)
- net B3_OSC_OUT: now reaches U8.9 (PF1-OSC_OUT)
- net B1_OSC_OUT: now reaches U1.6 (PH1)
Other:
- sheet Board1 ports: added MCU_OSC_OUT; removed none
- sheet Board2 ports: added MCU_OSC_OUT; removed none
- sheet Board3 ports: added MCU_OSC_OUT; removed none
Changed lines of the file:
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@@
 	(wire
 		(pts
+			(xy 146.05 184.15) (xy 147.32 184.15)
+		)
+		(stroke
+			(width 0)
+			(type default)
+		)
+	)
+	(wire
+		(pts
 			(xy 238.76 147.32) (xy 240.03 147.32)
 		)
@@
 	(wire
 		(pts
+			(xy 34.29 186.69) (xy 35.56 186.69)
+		)
+		(stroke
+			(width 0)
+			(type default)
+		)
+	)
+	(wire
+		(pts
 			(xy 69.85 167.64) (xy 68.58 167.64)
 		)
@@
 	(wire
 		(pts
+			(xy 224.79 57.15) (xy 241.3 57.15)
+		)
+		(stroke
+			(width 0)
+			(type default)
+		)
+	)
+	(wire
+		(pts
 			(xy 85.09 21.59) (xy 93.98 21.59)
 		)
@@
 	(wire
 		(pts
+			(xy 16.51 54.61) (xy 29.21 54.61)
+		)
+		(stroke
+			(width 0)
+			(type default)
+		)
+	)
+	(wire
+		(pts
 			(xy 113.03 170.18) (xy 114.3 170.18)
 		)
@@
 	(wire
 		(pts
-			(xy 34.29 187.96) (xy 35.56 187.96)
+			(xy 146.05 57.15) (xy 160.02 57.15)
+		)
+		(stroke
+			(width 0)
+			(type default)
+		)
+	)
+	(wire
+		(pts
+			(xy 34.29 190.5) (xy 35.56 190.5)
+		)
+		(stroke
+			(width 0)
+			(type default)
+		)
+	)
+	(wire
+		(pts
+			(xy 238.76 151.13) (xy 240.03 151.13)
 		)
 		(stroke
@@
 		)
 	)
+	(label "B1_OSC_OUT"
+		(at 34.29 186.69 180)
+		(effects
+			(font
+				(size 1.27 1.27)
+			)
+			(justify right bottom)
+		)
+	)
 	(label "SDIO_CK"
 		(at 16.51 95.25 0)
@@
 		)
 	)
+	(label "B1_OSC_OUT"
+		(at 16.51 54.61 0)
+		(effects
+			(font
+				(size 1.27 1.27)
+			)
+			(justify left bottom)
+		)
+	)
 	(label "B3_RS485_MCU_RX"
 		(at 162.56 87.63 0)
@@
 	)
 	(label "B1_USR_LED"
-		(at 34.29 187.96 180)
+		(at 34.29 190.5 180)
 		(effects
 			(font
@@
 		)
 	)
+	(label "B3_OSC_IN"
+		(at 241.3 54.61 180)
+		(effects
+			(font
+				(size 1.27 1.27)
+			)
+			(justify right bottom)
+		)
+	)
 	(label "LSM_CS"
 		(at 34.29 168.91 180)
@@
 		)
 	)
-	(label "B3_OSC_IN"
-		(at 241.3 54.61 180)
-		(effects
-			(font
-				(size 1.27 1.27)
-			)
-			(justify right bottom)
-		)
-	)
 	(label "B1_SWCLK"
 		(at 81.28 77.47 180)
@@
 		)
 	)
+	(label "B3_OSC_OUT"
+		(at 240.03 151.13 0)
+		(effects
+			(font
+				(size 1.27 1.27)
+			)
+			(justify left bottom)
+		)
+	)
+	(label "B2_OSC_OUT"
+		(at 160.02 57.15 180)
+		(effects
+			(font
+				(size 1.27 1.27)
+			)
+			(justify right bottom)
+		)
+	)
 	(label "GPIOB"
 		(at 95.25 95.25 0)
@@
 		)
 	)
+	(label "B2_OSC_OUT"
+		(at 147.32 184.15 0)
+		(effects
+			(font
+				(size 1.27 1.27)
+			)
+			(justify left bottom)
+		)
+	)
 	(label "B_CLK"
 		(at 92.71 77.47 0)
@@
 		)
 	)
+	(label "B3_OSC_OUT"
+		(at 241.3 57.15 180)
+		(effects
+			(font
+				(size 1.27 1.27)
+			)
+			(justify right bottom)
+		)
+	)
 	(label "B2_SWDIO"
 		(at 92.71 59.69 0)
@@
 		)
 		(pin "USR_LED" input
-			(at 35.56 187.96 180)
+			(at 35.56 190.5 180)
 			(effects
 				(font
@@
 			)
 		)
+		(pin "MCU_OSC_OUT" input
+			(at 35.56 186.69 180)
+			(effects
+				(font
+					(size 1.27 1.27)
+				)
+				(justify left)
+			)
+		)
 		(instances
 			(project "main"
@@
 			)
 		)
+		(pin "MCU_OSC_OUT" input
+			(at 146.05 184.15 0)
+			(effects
+				(font
+					(size 1.27 1.27)
+				)
+				(justify right)
+			)
+		)
 		(instances
 			(project "main"
@@
 			)
 		)
+		(pin "MCU_OSC_OUT" input
+			(at 238.76 151.13 0)
+			(effects
+				(font
+					(size 1.27 1.27)
+				)
+				(justify right)
+			)
+		)

Commit message: continue fixing chklst
Parts:
- added C22, C23, C31: 100n, Capacitor_SMD:C_0603_1608Metric, symbol Device:C_Small
- added R19: 10k, Resistor_SMD:R_0603_1608Metric, symbol Device:R
- added R21, R22, R23: 22, Resistor_SMD:R_0603_1608Metric, symbol Device:R
- added RN1: R_Net04_10k, Resistor_SMD:R_Array_Convex_4x0603, symbol Device:R_Network04
Connections:
- net +3V3: now also RN1.1 (common)
- net B1_NRST: now also C22.2
- net B2_CLK: now also R22.1; no longer U1.21 (PA5)
- net B2_MOSI: now also R21.2; no longer U1.23 (PA7)
- net B2_NRST: now also C23.1
- net B3_NRST: now also C31.1
- net B_MISO: now also R23.2; no longer U7.43 (PB4)
- net GND: now also C22.1, C23.2, C31.2, R19.1
- net SDIO_D0: now also RN1.5 (R4)
- net SDIO_D1: now also RN1.4 (R3)
- net SDIO_D2: now also RN1.3 (R2)
- net SDIO_D3: now also RN1.2 (R1)
- net at U1.60 (BOOT0): now also R19.2
- net GPS_SAFEBOOT: no longer names the net of U8.2 (PC14-OSC32_IN)
- new net: R22.2, U1.21 (PA5)
- new net: R23.1, U7.43 (PB4)
- new net: R21.1, U1.23 (PA7)
Other:
- sheet Board3 ports: added none; removed GPS_SAFEBOOT

Commit message: prep gerber and cpl/bom
Parts:
- removed RN1: R_Net04_10k, Resistor_SMD:R_Array_Convex_4x0603, symbol Device:R_Network04
- added RN1: 10k, Resistor_SMD:R_Array_Convex_4x0603, symbol Device:R_Pack04
- R21, R22, R23: LCSC (none) -> C23345
Connections:
- net +3V3: now also RN1.1 (R1.1), RN1.2 (R2.1), RN1.3 (R3.1), RN1.4 (R4.1)
- net SDIO_D0: now also RN1.8 (R1.2)
- net SDIO_D1: now also RN1.7 (R2.2)
- net SDIO_D2: now also RN1.6 (R3.2)
- net SDIO_D3: now also RN1.5 (R4.2)
Changed lines of the file:
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@@
 	(wire
 		(pts
+			(xy 88.9 194.31) (xy 91.44 194.31)
+		)
+		(stroke
+			(width 0)
+			(type default)
+		)
+	)
+	(wire
+		(pts
 			(xy 92.71 180.34) (xy 91.44 180.34)
 		)
@@
 	(wire
 		(pts
+			(xy 83.82 194.31) (xy 86.36 194.31)
+		)
+		(stroke
+			(width 0)
+			(type default)
+		)
+	)
+	(wire
+		(pts
 			(xy 34.29 161.29) (xy 35.56 161.29)
 		)
@@
 	(wire
 		(pts
+			(xy 86.36 194.31) (xy 88.9 194.31)
+		)
+		(stroke
+			(width 0)
+			(type default)
+		)
+	)
+	(wire
+		(pts
 			(xy 113.03 157.48) (xy 114.3 157.48)
 		)
@@
 			)
 		)
+		(property "LCSC" "C23345"
+			(at 74.93 54.61 0)
+			(hide yes)
+			(show_name no)
+			(do_not_autoplace no)
+			(effects
+				(font
+					(size 1.27 1.27)
+				)
+			)
+		)
 		(pin "1"
 		)
@@
 			)
 		)
+		(property "LCSC" "C23345"
+			(at 99.06 80.01 0)
+			(hide yes)
+			(show_name no)
+			(do_not_autoplace no)
+			(effects
+				(font
+					(size 1.27 1.27)
+				)
+			)
+		)
 		(pin "1"
 		)
@@
 			)
 		)
+		(property "LCSC" "C23345"
+			(at 74.93 59.69 0)
+			(hide yes)
+			(show_name no)
+			(do_not_autoplace no)
+			(effects
+				(font
+					(size 1.27 1.27)
+				)
+			)
+		)
 		(pin "1"
 		)
@@
 	)
 	(symbol
-		(lib_id "Device:C")
-		(at 85.09 25.4 0)
+		(lib_id "Device:R_Pack04")
+		(at 88.9 189.23 0)
 		(unit 1)
 		(body_style 1)
@@
 		(in_pos_files yes)
 		(dnp no)
-		(property "Reference" "C46"
-			(at 85.598 23.368 0)
+		(property "Reference" "RN1"
+			(at 96.52 187.96 0)
 			(show_name no)
 			(do_not_autoplace no)
@@
 					(size 1.27 1.27)
 				)
-				(justify left)
 			)
 		)
-		(property "Value" "100n"
-			(at 85.344 27.6861 0)
+		(property "Value" "10k"
+			(at 96.52 190.5 0)
 			(show_name no)
 			(do_not_autoplace no)
@@
 					(size 1.27 1.27)
 				)
-				(justify left)
 			)
 		)
-		(property "Footprint" "Capacitor_SMD:C_0603_1608Metric"
-			(at 86.0552 29.21 0)
+		(property "Footprint" "Resistor_SMD:R_Array_Convex_4x0603"
+			(at 88.9 189.23 0)
 			(hide yes)
 			(show_name no)
@@
 		)
 		(property "Datasheet" ""
-			(at 85.09 25.4 0)
+			(at 88.9 189.23 0)
 			(hide yes)
 			(show_name no)
@@
 			)
 		)
-		(property "Description" "Unpolarized capacitor"
-			(at 85.09 25.4 0)
+		(property "Description" "4 isolated 10k resistors (SD DAT0-3 pull-ups)"
+			(at 88.9 189.23 0)
+			(hide yes)
+			(show_name no)
+			(do_not_autoplace no)
+			(effects
+				(font
+					(size 1.27 1.27)
+				)
+			)
+		)
+		(property "LCSC" "C29718"
+			(at 88.9 189.23 0)
+			(hide yes)
+			(show_name no)
+			(do_not_autoplace no)
+			(effects
+				(font
+					(size 1.27 1.27)
+				)
+			)
+		)
+		(property "MPN" "UNI-ROYAL 4D03WGJ0103T5E"
+			(at 88.9 189.23 0)
 			(hide yes)
 			(show_name no)
@@
 		(pin "2"
 		)
+		(pin "3"
+		)
+		(pin "4"
+		)
+		(pin "5"
+		)
+		(pin "6"
+		)
+		(pin "7"
+		)
+		(pin "8"
+		)
 		(instances
 			(project "main"
 				(path "/6aa21aac-e8da-46e9-ae7a-f048cdfa6a26"
-					(reference "C46")
+					(reference "RN1")
 					(unit 1)
 				)
@@
 	)
 	(symbol
-		(lib_id "Device:R_Network04")
-		(at 86.36 189.23 180)
+		(lib_id "Device:C")
+		(at 85.09 25.4 0)
 		(unit 1)
 		(body_style 1)
@@
 		(in_pos_files yes)
 		(dnp no)
-		(fields_autoplaced yes)
-		(property "Reference" "RN1"
-			(at 93.98 187.7059 0)
+		(property "Reference" "C46"
+			(at 85.598 23.368 0)
 			(show_name no)
 			(do_not_autoplace no)
@@
 					(size 1.27 1.27)
 				)
-				(justify right)
+				(justify left)
 			)
 		)
-		(property "Value" "R_Net04_10k"
-			(at 93.98 190.2459 0)
+		(property "Value" "100n"
+			(at 85.344 27.6861 0)
 			(show_name no)
 			(do_not_autoplace no)
@@
 					(size 1.27 1.27)
 				)
-				(justify right)
+				(justify left)
 			)
 		)
-		(property "Footprint" "Resistor_SMD:R_Array_Convex_4x0603"
-			(at 79.375 189.23 90)
+		(property "Footprint" "Capacitor_SMD:C_0603_1608Metric"
+			(at 86.0552 29.21 0)
 			(hide yes)
 			(show_name no)
@@
 			)
 		)
-		(property "Datasheet" "http://www.vishay.com/docs/31509/csc.pdf"
-			(at 86.36 189.23 0)
+		(property "Datasheet" ""
+			(at 85.09 25.4 0)
 			(hide yes)
 			(show_name no)
@@
 			)
 		)
-		(property "Description" "4 resistor network, star topology, bussed resistors, small symbol"
-			(at 86.36 189.23 0)
+		(property "Description" "Unpolarized capacitor"
+			(at 85.09 25.4 0)
 			(hide yes)
 			(show_name no)
@@
 			)
 		)
-		(pin "4"
-		)
-		(pin "3"
+		(pin "1"
 		)
 		(pin "2"
 		)
-		(pin "5"
-		)
-		(pin "1"
-		)
 		(instances
 			(project "main"
 				(path "/6aa21aac-e8da-46e9-ae7a-f048cdfa6a26"
-					(reference "RN1")
+					(reference "C46")
 					(unit 1)
 				)
